File: X12 Power Distribuition.brd (EAGLE design)
At the start: 152.4 x 76.2 mm, 47 parts, among them Q1 SPB80P06P, Y1 ECS-80-S-4X

Commit message: fixed some erc warnings
Connections:
- removed net N$10: U$7.16
- removed net N$106: U$5.15
- removed net N$11: U$7.15
- removed net N$14: U$7.53
- removed net N$16: U$5.53
- removed net N$37: U$6.33
- removed net N$42: U$6.43
- removed net N$43: U$6.45
- removed net N$77: U$6.34
- removed net N$82: U$6.44
- removed net N$83: U$6.46
- removed net N$85: U$5.2
- removed net N$9: U$7.2
- removed net N$92: U$5.16

Commit message: more modifications
Parts:
- moved C6 11.3 mm to (123.2, 42.7), turned to 270 degrees
- moved C5 11.1 mm to (126.0, 42.7), turned to 270 degrees
- moved R7 3.24 mm to (118.8, 43.7), flipped to the bottom
- moved R5 3.24 mm to (122.0, 43.8), flipped to the bottom
- moved C1 2.62 mm to (125.4, 49.0)
- moved C3 2.62 mm to (122.7, 48.9)
- moved C4 0.90 mm to (140.6, 39.5)
- moved C2 0.64 mm to (137.6, 39.8)
- moved C7 0.63 mm to (128.8, 53.4)
- moved R6 0.63 mm to (131.9, 53.6)
- moved R8 0.63 mm to (135.3, 53.5)
Routing:
- net +3V3: track 141.6 -> 136.6 mm
- net OSC_IN: track 6.67 -> 10.1 mm, vias 0 -> 1
- net OSC_OUT: track 3.18 -> 6.62 mm, vias 0 -> 1
- net N$7: track 18.9 -> 21.6 mm
- net N$6: track 19.5 -> 22.0 mm
- net 3V3GND: track 154.6 -> 155.7 mm
- net NRST: track 52.9 -> 53.8 mm
- net LED: track 4.23 -> 3.59 mm

Commit message: Small edits on board
Added Labels
Parts:
- moved H1 1.42 mm to (4.01, 4.11)
- moved H4 1.27 mm to (148.4, 72.3)
- moved H3 0.90 mm to (4.24, 72.3)
Other:
- board text added: "48V INPUT"
- board text added: "48V POE"
- board text added: "BRICK A CONNECTOR"
- board text added: "BRICK B CONNECTOR"
- board text added: "CONVERSION CONNECTOR"
- board text added: "Pin 1"
